File: PCB/easybutton.kicad_pcb (KiCad board)
At the start: 2 copper layers, 30.5 x 57.2 mm, 9 parts, among them SW1 Speaker button, U1 NodeMCU1.0(ESP-12E)

Commit message: Updating PCB and readme
Other:
- board text added: "Align controller to this side"
